File: analog_dice.kicad_pcb (KiCad board)
At the start: 2 copper layers, 35 x 35 mm, 32 parts, among them Q1 2SA1774T1G, SW1 SW_SPST, SW2 4081 Vibration Switch, U1 LMC555xM, U2 74HC4017PW, U3 74LCX32FT, U4 74LCX32FT

Commit message: fix
Parts:
- Q1: value 2SA1774T1G -> MMBT5401T; footprint Package_TO_SOT_SMD:SOT-416 -> Package_TO_SOT_SMD:SOT-523
- SW1: footprint Button_Switch_SMD:SW_DIP_SPSTx01_Slide_Copal_CHS-01A_W5.08mm_P1.27mm_JPin -> Button_Switch_SMD:SW_DIP_SPSTx01_Slide_Copal_CHS-01B_W7.62mm_P1.27mm; moved to F.Cu
- moved SW1 31.8 mm to (92.5, 61.8), turned to 180 degrees
- renumbered C5 to C1, C4 to C2, C1 to C4, C2 to C5, D7 to D2, D5 to D3, D6 to D4, D2 to D5, D4 to D6, D3 to D7, R2 to R1, R1 to R10, R10 to R2, R6 to R4, R7 to R5, R8 to R6, R4 to R7, R9 to R8, R5 to R9, U3 to U1, U4 to U2, U1 to U3, U2 to U4
Routing:
- net Net-(BT1-+): track 65.1 -> 45.5 mm, vias 0 -> 1
- net +3.3V: track 40.6 -> 54.4 mm
Other:
- board text added: "Designed By: Kyle Schmerge Revision 1.0"
- board text added: "Fully Discrete Electronic Die"
- board text added: "Power"
