File: analog_dice.kicad_pcb (KiCad board)
At the start: 2 copper layers, 35 x 35 mm, 32 parts, among them Q1 MMBT5401T, SW1 SW_SPST, SW2 4081 Vibration Switch, U1 74LCX32FT, U2 74LCX32FT, U3 LMC555xM, U4 74HC4017PW

Commit message: fix
Routing:
- net +3.3V: track 54.4 -> 58.9 mm, vias 8 -> 9
- net Net-(BT1-+): track 45.5 -> 43.2 mm
Changed lines of the file:
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@@
 		(attr smd)
 		(fp_line
-			(start 10.922 5.08)
-			(end 8.382 7.62)
+			(start 9.906 5.08)
+			(end 7.366 7.62)
 			(stroke
 				(width 0.1)
@@
 		)
 		(fp_line
-			(start 10.922 -5.08)
-			(end 10.922 5.08)
+			(start 9.906 3)
+			(end 9.906 5.08)
 			(stroke
 				(width 0.1)
@@
 		)
 		(fp_line
-			(start 8.382 7.62)
-			(end 5.08 7.62)
+			(start 7.366 7.62)
+			(end 4.064 7.62)
 			(stroke
 				(width 0.1)
@@
 		)
 		(fp_line
-			(start -8.382 7.62)
-			(end -5.08 7.62)
+			(start -6.604 7.62)
+			(end -4.064 7.62)
 			(stroke
 				(width 0.1)
@@
 		)
 		(fp_line
-			(start -10.922 5.08)
-			(end -8.382 7.62)
+			(start -9.144 5.08)
+			(end -6.604 7.62)
 			(stroke
 				(width 0.1)
@@
 		)
 		(fp_line
-			(start -10.922 -5.08)
-			(end -10.922 5.08)
+			(start -9.144 3)
+			(end -9.144 5.08)
 			(stroke
 				(width 0.1)
@@
 		)
 		(fp_line
-			(start 14.224 2.794)
-			(end 14.224 -2.794)
+			(start 11.9634 2.794)
+			(end 11.9634 -2.794)
 			(stroke
 				(width 0.05)
@@
 		)
 		(fp_line
-			(start 14.224 -2.794)
-			(end 11.176 -2.794)
+			(start 11.9634 -2.794)
+			(end 8.8138 -2.794)
 			(stroke
 				(width 0.05)
@@
 		)
 		(fp_line
-			(start 11.176 10.16)
-			(end -11.176 10.16)
+			(start 8.8138 10.16)
+			(end -8.8138 10.16)
 			(stroke
 				(width 0.05)
@@
 		)
 		(fp_line
-			(start 11.176 2.794)
-			(end 14.224 2.794)
+			(start 8.8138 2.794)
+			(end 11.9634 2.794)
 			(stroke
 				(width 0.05)
@@
 		)
 		(fp_line
-			(start 11.176 2.794)
-			(end 11.176 10.16)
+			(start 8.8138 2.794)
+			(end 8.8138 10.16)
 			(stroke
 				(width 0.05)
@@
 		)
 		(fp_line
-			(start 11.176 -2.794)
-			(end 11.176 -10.16)
+			(start 8.8138 -2.794)
+			(end 8.8138 -10.16)
 			(stroke
 				(width 0.05)
@@
 		)
 		(fp_line
-			(start -11.176 2.794)
-			(end -11.176 10.16)
+			(start -8.8138 2.794)
+			(end -8.8138 10.16)
 			(stroke
 				(width 0.05)
@@
 		)
 		(fp_line
-			(start -11.176 -2.794)
-			(end -11.176 -10.16)
+			(start -8.8138 -2.794)
+			(end -8.8138 -10.16)
 			(stroke
 				(width 0.05)
@@
 		)
 		(fp_line
-			(start -11.176 -10.16)
-			(end 11.176 -10.16)
+			(start -8.8138 -10.16)
+			(end 8.8138 -10.16)
 			(stroke
 				(width 0.05)
@@
 		)
 		(fp_line
-			(start -14.224 2.794)
-			(end -11.176 2.794)
+			(start -11.9634 2.794)
+			(end -8.8138 2.794)
 			(stroke
 				(width 0.05)
@@
 		)
 		(fp_line
-			(start -14.224 2.794)
-			(end -14.224 -2.794)
+			(start -11.9634 2.794)
+			(end -11.9634 -2.794)
 			(stroke
 				(width 0.05)
@@
 		)
 		(fp_line
-			(start -14.224 -2.794)
-			(end -11.176 -2.794)
+			(start -11.9634 -2.794)
+			(end -8.8138 -2.794)
 			(stroke
 				(width 0.05)
@@
 		)
 		(pad "1" smd rect
-			(at -12.7 0 180)
+			(at -10.5 0 180)
 			(size 2.54 5.08)
 			(layers "B.Cu" "B.Mask" "B.Paste")
@@
 		)
 		(pad "1" smd rect
-			(at 12.7 0 180)
+			(at 10.5 0 180)
 			(size 2.54 5.08)
 			(layers "B.Cu" "B.Mask" "B.Paste")
@@
 		(pad "2" smd circle
 			(at 0 0 180)
-			(size 17.78 17.78)
+			(size 17 17)
 			(layers "B.Cu" "B.Mask" "B.Paste")
 			(net 2 "GND")
@@
 	)
 	(segment
-		(start 84 64.25)
-		(end 101 64.25)
+		(start 83.525 63.725)
+		(end 101.525 63.725)
 		(width 0.2)
 		(layer "B.Cu")
@@
 	)
 	(segment
-		(start 79.8 54.75)
-		(end 79.8 60.05)
+		(start 103 62.25)
+		(end 101.525 63.725)
 		(width 0.2)
 		(layer "B.Cu")
@@
 	)
 	(segment
-		(start 101 64.25)
-		(end 105.2 60.05)
+		(start 82 62.2)
+		(end 83.525 63.725)
 		(width 0.2)
 		(layer "B.Cu")
@@
 	)
 	(segment
-		(start 79.8 60.05)
-		(end 84 64.25)
+		(start 82 54.75)
+		(end 82 62.2)
 		(width 0.2)
 		(layer "B.Cu")
@@
 	)
 	(segment
-		(start 105.2 60.05)
-		(end 105.2 54.75)
+		(start 103 54.75)
+		(end 103 62.25)
 		(width 0.2)
 		(layer "B.Cu")
@@
 	)
 	(segment
+		(start 101.47 59.25)
+		(end 104.02 61.8)
+		(width 0.2)
+		(layer "F.Cu")
+		(net 5)
+	)
+	(segment
 		(start 100.67 44)
 		(end 98.63 46.04)
@@
 	)
 	(segment
+		(start 104.02 61.8)
+		(end 104.9 61.8)
+		(width 0.2)
+		(layer "F.Cu")
+		(net 5)
+	)
+	(segment
 		(start 108.1 38.43)
 		(end 106.1 36.43)
@@
 		(net 5)
 	)
+	(via
+		(at 104.9 61.8)
+		(size 0.6)
+		(drill 0.3)
+		(layers "F.Cu" "B.Cu")
+		(net 5)
+	)
